Commit message: added ankles to improve standing

File: models/biped.urdf (robot description, URDF)
Before this commit: robot simple_biped, 5 links, 4 joints
Links:
- added link left_foot, mass 1; collision box size=0.18 0.08 0.04; visual box size=0.18 0.08 0.04
- added link right_foot, mass 1; collision box size=0.18 0.08 0.04; visual box size=0.18 0.08 0.04
Joints:
- added joint left_ankle: type revolute, parent left_shin, child left_foot, origin xyz=0 0 -0.3, axis 0 1 0, limit lower=-0.6 upper=0.6 effort=80
- added joint right_ankle: type revolute, parent right_shin, child right_foot, origin xyz=0 0 -0.3, axis 0 1 0, limit lower=-0.6 upper=0.6 effort=80
- joint left_hip: limit lower=-1.5 upper=1.5 effort=100 -> lower=-1.5 upper=1.5 effort=120
- joint left_knee: limit lower=-1.5 upper=0.0 effort=100 -> lower=-1.5 upper=0.0 effort=120
- joint right_hip: limit lower=-1.5 upper=1.5 effort=100 -> lower=-1.5 upper=1.5 effort=120
- joint right_knee: limit lower=-1.5 upper=0.0 effort=100 -> lower=-1.5 upper=0.0 effort=120

Commit message: improve model for standing

File: models/biped.urdf (robot description, URDF)
Before this commit: robot simple_biped, 7 links, 6 joints
Links:
- link left_foot: mass 1 -> 2.0; geometry collision box size=0.26 0.12 0.05; visual box size=0.26 0.12 0.05
- link left_shin: mass 2 -> 2.8; geometry collision capsule length=0.32 radius=0.04; visual capsule length=0.32 radius=0.04
- link left_thigh: mass 3 -> 3.5; geometry collision capsule length=0.32 radius=0.045; visual capsule length=0.32 radius=0.045
- link right_foot: mass 1 -> 2.0; geometry collision box size=0.26 0.12 0.05; visual box size=0.26 0.12 0.05
- link right_shin: mass 2 -> 2.8; geometry collision capsule length=0.32 radius=0.04; visual capsule length=0.32 radius=0.04
- link right_thigh: mass 3 -> 3.5; geometry collision capsule length=0.32 radius=0.045; visual capsule length=0.32 radius=0.045
- link torso: mass 10 -> 12; geometry collision box size=0.25 0.14 0.45; visual box size=0.25 0.14 0.45
Joints:
- joint left_ankle: limit lower=-0.6 upper=0.6 effort=80 -> lower=-0.45 upper=0.45; origin xyz=0 0 -0.3 -> xyz=0 0 -0.32
- joint left_hip: limit lower=-1.5 upper=1.5 effort=120 -> lower=-1.2 upper=1.2 effort=180; origin xyz=0 0.08 -0.2 -> xyz=0 0.11 -0.25
- joint left_knee: limit lower=-1.5 upper=0.0 effort=120 -> lower=-1.0 upper=-0.05; origin xyz=0 0 -0.3 -> xyz=0 0 -0.32
- joint right_ankle: limit lower=-0.6 upper=0.6 effort=80 -> lower=-0.45 upper=0.45; origin xyz=0 0 -0.3 -> xyz=0 0 -0.32
- joint right_hip: limit lower=-1.5 upper=1.5 effort=120 -> lower=-1.2 upper=1.2 effort=180; origin xyz=0 -0.08 -0.2 -> xyz=0 -0.11 -0.25
- joint right_knee: limit lower=-1.5 upper=0.0 effort=120 -> lower=-1.0 upper=-0.05; origin xyz=0 0 -0.3 -> xyz=0 0 -0.32
